Commit message: updated to run with MiR

File: ur_description/urdf/inc/ur_macro.xacro (robot description, xacro)
@@ -64,6 +64,6 @@
     <xacro:ur_arm_transmission prefix="${prefix}" hw_interface="${transmission_hw_interface}" />
     <!-- links: main serial chain -->
-    <link name="${prefix}base_link"/>
-    <link name="${prefix}base_link_inertia">
+    <link name="${prefix}base_link_ur10"/>
+    <link name="${prefix}base_link_ur10_inertia">
       <visual>
         <origin xyz="0 0 0" rpy="0 0 ${pi}"/>
@@ -207,10 +207,10 @@
     </link>
     <!-- joints: main serial chain -->
-    <joint name="${prefix}base_link-base_link_inertia" type="fixed">
-      <parent link="${prefix}base_link" />
-      <child link="${prefix}base_link_inertia" />
-      <!-- 'base_link' is REP-103 aligned (so X+ forward), while the internal
+    <joint name="${prefix}base_link_ur10-base_link_ur10_inertia" type="fixed">
+      <parent link="${prefix}base_link_ur10" />
+      <child link="${prefix}base_link_ur10_inertia" />
+      <!-- 'base_link_ur10' is REP-103 aligned (so X+ forward), while the internal
            frames of the robot/controller have X+ pointing backwards.
-           Use the joint between 'base_link' and 'base_link_inertia' (a dummy
+           Use the joint between 'base_link_ur10' and 'base_link_ur10_inertia' (a dummy
            link/frame) to introduce the necessary rotation over Z (of pi rad).
       -->
@@ -218,5 +218,5 @@
     </joint>
     <joint name="${prefix}shoulder_pan_joint" type="revolute">
-      <parent link="${prefix}base_link_inertia" />
+      <parent link="${prefix}base_link_ur10_inertia" />
       <child link="${prefix}shoulder_link" />
       <origin xyz="${shoulder_x} ${shoulder_y} ${shoulder_z}" rpy="${shoulder_roll} ${shoulder_pitch} ${shoulder_yaw}" />
@@ -289,8 +289,8 @@
       <dynamics damping="0" friction="0"/>
     </joint>
-    <!-- ROS-Industrial 'base' frame: base_link to UR 'Base' Coordinates transform -->
+    <!-- ROS-Industrial 'base' frame: base_link_ur10 to UR 'Base' Coordinates transform -->
     <link name="${prefix}base"/>
-    <joint name="${prefix}base_link-base_fixed_joint" type="fixed">
-      <!-- Note the rotation over Z of pi radians: as base_link is REP-103
+    <joint name="${prefix}base_link_ur10-base_fixed_joint" type="fixed">
+      <!-- Note the rotation over Z of pi radians: as base_link_ur10 is REP-103
            aligned (ie: has X+ forward, Y+ left and Z+ up), this is needed
            to correctly align 'base' with the 'Base' coordinate system of
@@ -298,5 +298,5 @@
       -->
       <origin xyz="0 0 0" rpy="0 0 ${pi}"/>
-      <parent link="${prefix}base_link"/>
+      <parent link="${prefix}base_link_ur10"/>
       <child link="${prefix}base"/>
     </joint>
